File: Code/CoverLayerOutput.brd (EAGLE design)
At the start: 420.5 x 1359.5 mm, 0 parts

Commit message: Attempt 2, removal of Plain
Other:
- board size 420.5 x 1359.5 mm -> 160 x 100 mm
Changed lines of the file:
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@@
 </pass>
 </autorouter>
-<plain>
-<wire x1="0" y1="0" x2="420.5" y2="0" width="0" layer="20"/>
-<wire x1="420.5" y1="0" x2="420.5" y2="1359.52" width="0" layer="20"/>
-<wire x1="420.5" y1="1359.52" x2="0" y2="1359.52" width="0" layer="20"/>
-<wire x1="0" y1="1359.52" x2="0" y2="0" width="0" layer="20"/>
-<rectangle x1="0" y1="0" x2="420.5" y2="10.5" layer="29"/>
-<rectangle x1="0" y1="25.3" x2="420.5" y2="29.3" layer="29"/>
-<rectangle x1="0" y1="44.1" x2="420.5" y2="48.1" layer="29"/>
-<rectangle x1="0" y1="62.9" x2="420.5" y2="66.9" layer="29"/>
-<rectangle x1="0" y1="81.7" x2="420.5" y2="1359.52" layer="29"/>
-</plain>
 <signals>
 <signal name="PAD$A0">
