File: Code/CoverLayerOutput.brd (EAGLE design)
At the start: 160 x 100 mm, 0 parts

Commit message: updates
new origins, correct segment measurments, and other stuff
Other:
- board size 160 x 100 mm -> 711 x 170 mm
