File: CoverLayerOutput.brd (EAGLE design)
At the start: 420.5 x 1359.5 mm, 0 parts

Commit message: forgot stuff
Forgot to have the last x change
Other:
- board size 420.5 x 1359.5 mm -> 160 x 100 mm
